Commit message: update README, clean code

File: BimanGrasp-Optimization/mjcf/dual_ur5_shadow/dual_ur5_shadow.urdf (robot description, URDF)
Before this commit: robot dual_ur5, 72 links, 71 joints
Links:
- link lh_ffdistal: geometry visual mesh filename=./shadow/stl/f_distal_pst.stl
- link lh_ffknuckle: geometry visual mesh filename=./shadow/stl/f_knuckle.stl
- link lh_ffmiddle: geometry visual mesh filename=./shadow/stl/f_middle.stl
- link lh_ffproximal: geometry visual mesh filename=./shadow/stl/f_proximal.stl
- link lh_lfdistal: geometry visual mesh filename=./shadow/stl/f_distal_pst.stl
- link lh_lfknuckle: geometry visual mesh filename=./shadow/stl/f_knuckle.stl
- link lh_lfmetacarpal: geometry visual mesh filename=./shadow/stl/left_lf_metacarpal.stl
- link lh_lfmiddle: geometry visual mesh filename=./shadow/stl/f_middle.stl
- link lh_lfproximal: geometry visual mesh filename=./shadow/stl/f_proximal.stl
- link lh_mfdistal: geometry visual mesh filename=./shadow/stl/f_distal_pst.stl
- link lh_mfknuckle: geometry visual mesh filename=./shadow/stl/f_knuckle.stl
- link lh_mfmiddle: geometry visual mesh filename=./shadow/stl/f_middle.stl
- link lh_mfproximal: geometry visual mesh filename=./shadow/stl/f_proximal.stl
- link lh_palm: geometry visual mesh filename=./shadow/stl/left_palm.stl
- link lh_rfdistal: geometry visual mesh filename=./shadow/stl/f_distal_pst.stl
- link lh_rfknuckle: geometry visual mesh filename=./shadow/stl/f_knuckle.stl
- link lh_rfmiddle: geometry visual mesh filename=./shadow/stl/f_middle.stl
- link lh_rfproximal: geometry visual mesh filename=./shadow/stl/f_proximal.stl
- link lh_thdistal: geometry visual mesh filename=./shadow/stl/th_distal_pst.stl
- link lh_thmiddle: geometry visual mesh filename=./shadow/stl/th_middle.stl
- link lh_thproximal: geometry visual mesh filename=./shadow/stl/th_proximal.stl
- link rh_ffdistal: geometry visual mesh filename=./shadow/stl/f_distal_pst.stl
- link rh_ffknuckle: geometry visual mesh filename=./shadow/stl/f_knuckle.stl
- link rh_ffmiddle: geometry visual mesh filename=./shadow/stl/f_middle.stl
- link rh_ffproximal: geometry visual mesh filename=./shadow/stl/f_proximal.stl
- link rh_lfdistal: geometry visual mesh filename=./shadow/stl/f_distal_pst.stl
- link rh_lfknuckle: geometry visual mesh filename=./shadow/stl/f_knuckle.stl
- link rh_lfmetacarpal: geometry visual mesh filename=./shadow/stl/right_lf_metacarpal.stl
- link rh_lfmiddle: geometry visual mesh filename=./shadow/stl/f_middle.stl
- link rh_lfproximal: geometry visual mesh filename=./shadow/stl/f_proximal.stl
- link rh_mfdistal: geometry visual mesh filename=./shadow/stl/f_distal_pst.stl
- link rh_mfknuckle: geometry visual mesh filename=./shadow/stl/f_knuckle.stl
- link rh_mfmiddle: geometry visual mesh filename=./shadow/stl/f_middle.stl
- link rh_mfproximal: geometry visual mesh filename=./shadow/stl/f_proximal.stl
- link rh_palm: geometry visual mesh filename=./shadow/stl/right_palm.stl
- link rh_rfdistal: geometry visual mesh filename=./shadow/stl/f_distal_pst.stl
- link rh_rfknuckle: geometry visual mesh filename=./shadow/stl/f_knuckle.stl
- link rh_rfmiddle: geometry visual mesh filename=./shadow/stl/f_middle.stl
- link rh_rfproximal: geometry visual mesh filename=./shadow/stl/f_proximal.stl
- link rh_thdistal: geometry visual mesh filename=./shadow/stl/th_distal_pst.stl
- link rh_thmiddle: geometry visual mesh filename=./shadow/stl/th_middle.stl
- link rh_thproximal: geometry visual mesh filename=./shadow/stl/th_proximal.stl
